File: pcb/tophat.brd (EAGLE design)
At the start: 100 x 76 mm, 11 parts

Commit message: 3-3-22 Updates
Parts:
- added C1, C2: (no value), rcl:E5-10,5
- added JP4, JP7: (no value), pinhead:1X07
- added JP5: (no value), pinhead:1X02
- added JP6: (no value), pinhead:1X04
- added JP8: PWR_CONN, railbaron:PWR_CONN
- added JP9: (no value), pinhead:2X03
- added R6, R7: (no value), rcl:0207/10
- added SJ1, SJ2: (no value), jumper:SJ_2
- added TP1, TP10, TP11, TP12, TP13, TP2, TP3, TP4, TP5, TP6, TP7, TP8, TP9: TPB2,54, testpad:B2,54
- U$1: device teensy4_fewerpins:TEENSY_4.0 -> railbaron:TEENSY_4.0
- moved U$2 8.51 mm to (28.6, 60.3)
- moved R5 8.13 mm to (10.1, 12.3), turned to 0 degrees
- moved R1 7.72 mm to (10.1, 14.9), turned to 0 degrees
- moved R4 6.15 mm to (10.1, 4.35), turned to 0 degrees
- moved R3 2.20 mm to (10.1, 6.97), turned to 0 degrees
- moved R2 1.89 mm to (10.1, 9.59), turned to 0 degrees
- moved U$3 1.40 mm to (53.1, 60.5)
- moved JP2 0.13 mm to (0.91, 38.0)
Connections:
- removed net N$3: JP1.8, U$1.0/RX
- new net BCLK: JP1.12, JP4.6, TP7.TP
- new net CS0: JP1.24, JP7.5
- new net CS1: JP1.26, JP7.6
- new net I2SD: JP1.40, JP4.5, TP8.TP
- new net LRCLK: JP1.35, JP4.7, TP6.TP
- new net MISO: JP1.21, JP7.3
- new net MOSI: JP1.19, JP7.2
- new net N$20: JP4.4, R6.1, SJ2.2
- new net N$21: R6.2, SJ1.2
- new net PI>T: JP1.8, TP9.TP, U$1.0/RX
- new net SCL: JP1.5, JP6.3
- new net SDA: JP1.3, JP6.2
- new net SPI_CLK: JP1.23, JP7.4
- new net T>PI: JP1.10, TP10.TP, U$1.1/TX
- net +3V3: now also TP12.TP
- net +5V: now also C1.+, C2.+, JP2.12, JP2.16, JP2.4, JP2.8, JP4.1, JP5.1, JP6.1, JP7.1, JP8.P$2, JP9.1, JP9.3, JP9.5, SJ1.3, SJ2.1, TP11.TP; no longer JP2.1, JP2.13, JP2.5, JP2.9
- net CLK: now also TP1.TP, U$1.12/MISO; no longer U$1.10/CS
- net DATA: now also TP5.TP, U$1.9/CS; no longer U$1.12/MISO
- net GND: now also C1.-, C2.-, JP2.11, JP2.15, JP2.3, JP2.7, JP4.2, JP5.2, JP6.4, JP7.7, JP8.P$1, JP9.2, JP9.4, JP9.6, R7.2, SJ1.1, SJ2.3, TP13.TP; no longer JP2.10, JP2.14, JP2.2, JP2.6, U$2.13, U$3.13
- net LATCH: now also TP3.TP, U$1.11/MOSI; no longer U$1.9/CS
- net LED_CLK: now also JP2.1, JP2.13, JP2.5, JP2.9; no longer JP2.12, JP2.16, JP2.4, JP2.8
- net LED_DIO1: now also JP2.2; no longer JP2.3
- net LED_DIO2: now also JP2.6; no longer JP2.7
- net LED_DIO3: now also JP2.10; no longer JP2.11
- net LED_DIO4: now also JP2.14; no longer JP2.15
- net N$1: now also TP4.TP
- net N$10: now also U$2.1; no longer U$2.2
- net N$2: now also JP1.37, U$1.ON/OFF; no longer JP1.10, U$1.1/TX
- net N$9: now also U$2.2; no longer U$2.1
- net RESET: now also JP1.7, R7.1, TP2.TP, U$1.10/CS, U$2.13, U$3.13; no longer U$1.11/MOSI
Routing:
- net I2SD: track 0.00 -> 111.1 mm
- net LRCLK: track 0.00 -> 92.4 mm
- net RESET: track 29.9 -> 120.0 mm, vias 2 -> 3
- net BCLK: track 0.00 -> 68.8 mm
- net T>PI: track 0.00 -> 55.9 mm
- net PI>T: track 0.00 -> 48.0 mm
- net N$3: track 45.2 -> 0.00 mm
- net GND: track 6.46 -> 36.9 mm, vias 4 -> 5
- net LED_CLK: track 76.2 -> 50.8 mm
- net N$20: track 0.00 -> 18.3 mm
- net +5V: track 0.00 -> 17.8 mm
- net N$9: track 24.9 -> 9.68 mm
- net N$1: track 24.9 -> 39.9 mm
- net LATCH: track 36.4 -> 49.4 mm, vias 0 -> 1
- net LED_DIO1: track 32.6 -> 22.3 mm
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Other:
- board size 100 x 76 mm -> 89.4 x 76 mm
- board text added: "- +"
- board text added: "12dB"
- board text added: "15dB"
- board text added: "3V3"
- board text added: "3dB"
- board text added: "5V"
- board text added: "6dB"
- board text added: "BCLK"
- board text added: "C"
- board text added: "CLK"
- board text added: "CS0"
- board text added: "CS1"
- board text added: "D"
- board text added: "DC"
- board text added: "GND"
- board text added: "I2SD"
- board text added: "L"
- board text added: "LRCLK"
- board text added: "MISO"
- board text added: "MOSI"
- board text added: "R"
- board text added: "RAIL BARON HAT BRIAN BOUCHER Rev A, Feb 2022"
- board text added: "SCL"
- board text added: "SDA"
- board text added: "T>π"
- board text added: "π>T"
