File: pcb/tophat.sch (EAGLE design)
At the start: 11 parts

Commit message: 3-3-22 Updates
Parts:
- added C1, C2: (no value), rcl:CPOL-USE5-10.5
- added JP4, JP7: (no value), pinhead:PINHD-1X7
- added JP5: (no value), pinhead:PINHD-1X2
- added JP6: (no value), pinhead:PINHD-1X4
- added JP8: PWR_CONN, railbaron:PWR_CONN
- added JP9: (no value), pinhead:PINHD-2X3
- added R6, R7: (no value), rcl:R-US_0207/10
- added SJ1, SJ2: (no value), jumper:SJ2W
- added TP1, TP10, TP11, TP12, TP13, TP2, TP3, TP4, TP5, TP6, TP7, TP8, TP9: TPB2,54, testpad:TPB2,54
- U$1: device teensy4_fewerpins:TEENSY_4.0 -> railbaron:TEENSY_4.0
Connections:
- removed net N$3: JP1.8, U$1.0/RX1
- new net BCLK: JP1.12, JP4.6, TP7.TP
- new net CS0: JP1.24, JP7.5
- new net CS1: JP1.26, JP7.6
- new net I2SD: JP1.40, JP4.5, TP8.TP
- new net LRCLK: JP1.35, JP4.7, TP6.TP
- new net MISO: JP1.21, JP7.3
- new net MOSI: JP1.19, JP7.2
- new net N$20: JP4.4, R6.1, SJ2.2
- new net N$21: R6.2, SJ1.2
- new net PI>T: JP1.8, TP9.TP, U$1.0/RX1
- new net SCL: JP1.5, JP6.3
- new net SDA: JP1.3, JP6.2
- new net SPI_CLK: JP1.23, JP7.4
- new net T>PI: JP1.10, TP10.TP, U$1.1/TX1
- net +3V3: now also TP12.TP
- net +5V: now also C1.+, C2.+, JP2.12, JP2.16, JP2.4, JP2.8, JP4.1, JP5.1, JP6.1, JP7.1, JP8.POS, JP9.1, JP9.3, JP9.5, SJ1.3, SJ2.1, TP11.TP; no longer JP2.1, JP2.13, JP2.5, JP2.9
- net CLK: now also TP1.TP, U$1.12/MISO, U$2.SRCLK, U$3.SRCLK; no longer U$1.10/CS, U$2.SHCP, U$3.SHCP
- net DATA: now also TP5.TP, U$1.9, U$2.SER; no longer U$1.12/MISO, U$2.DS
- net GND: now also C1.-, C2.-, JP2.11, JP2.15, JP2.3, JP2.7, JP4.2, JP5.2, JP6.4, JP7.7, JP8.NEG, JP9.2, JP9.4, JP9.6, R7.2, SJ1.1, SJ2.3, TP13.TP; no longer JP2.10, JP2.14, JP2.2, JP2.6, U$2./OE, U$3./OE
- net LATCH: now also TP3.TP, U$1.11/MOSI, U$2.RCLK, U$3.RCLK; no longer U$1.9, U$2.STCP, U$3.STCP
- net LED_CLK: now also JP2.1, JP2.13, JP2.5, JP2.9; no longer JP2.12, JP2.16, JP2.4, JP2.8
- net LED_DIO1: now also JP2.2; no longer JP2.3
- net LED_DIO2: now also JP2.6; no longer JP2.7
- net LED_DIO3: now also JP2.10; no longer JP2.11
- net LED_DIO4: now also JP2.14; no longer JP2.15
- net N$1: now also TP4.TP, U$3.SER; no longer U$3.DS
- net N$10: now also U$2.Q1; no longer U$2.Q2
- net N$2: now also JP1.37, U$1.ON/OFF; no longer JP1.10, U$1.1/TX1
- net N$9: now also U$2.Q2; no longer U$2.Q1
- net RESET: now also JP1.7, R7.1, TP2.TP, U$1.10/CS, U$2./RCLR, U$2./SRCLR, U$3./RCLR, U$3./SRCLR; no longer U$1.11/MOSI, U$2./MR, U$3./MR
Other:
- moved on the sheet: JP3
